File: modules/sliders/hardware/sliders.kicad_sch (KiCad schematic)
At the start: 8 parts, among them J5 Button, SW2 SW_Push

Commit message: Modified Slider PCB Design
Parts:
- A1: footprint Module:RaspberryPi_Pico_Common_THT -> Module:RaspberryPi_Pico_Common_THT_no_antenna
Changed lines of the file:
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@@
 			)
 		)
-		(property "Footprint" "Module:RaspberryPi_Pico_Common_THT"
+		(property "Footprint" "Module:RaspberryPi_Pico_Common_THT_no_antenna"
 			(at 115.57 139.7 0)
 			(hide yes)
